File: schematic/_autosave-_autosave-_autosave-Test1Kicad.kicad_sch (KiCad schematic)
At the start: 72 parts, among them IC1 BMI055, J1 Power Module 1, J10 CAP & ADC IN, J11 SPI Port, J12 I2C A, J13 FMU PWM OUT, J14 PPM RC, J15 2908-05WB-MG, J2 Power Module 2, J3 USB, J4 Telemetry 1, J5 Telemetry 2, J6 UART & I2C B, J7 CAN 1, J8 CAN 2, J9 GPS Module, U1 STM32F765IIKx, U10 TJA1051TK-3, U11 LT3080xDD, U2 NEO-M8N, U3 IST8310, U4 ICM-20602, U5 ICM-20689, U6 MS5611-01BA, U7 LT3080xDD, U8 STM32F103V8Tx, U9 TJA1051TK-3, Y1 ABM2-8.000MHZ-D4Y-T

Commit message: Few Ports
Parts:
- removed C16: 2.2uF, symbol Device:C_Small
- removed C17: 1uf, symbol Device:C_Small
- removed U2: NEO-M8N, RF_GPS:ublox_NEO, symbol RF_GPS:NEO-M8N
- removed U7: LT3080xDD, Package_DFN_QFN:DFN-8-1EP_3x3mm_P0.5mm_EP1.66x2.38mm, symbol Regulator_Linear:LT3080xDD
- added C28, C29: 1uf, symbol Device:C_Small
- added J16: RC, symbol Connector:Conn_01x05_Socket
- added J17: SBUS, symbol Connector:Conn_01x03_Socket
- added U12: LP5907MFX-3.3, Package_TO_SOT_SMD:SOT-23-5, symbol Regulator_Linear:LP5907MFX-3.3
- R1: value 330k -> 10K
Connections:
- net GND: now also J9.10 (Pin_10), U4.8 (FSYNC), C28.2, C29.2, J16.5 (Pin_5), J17.3 (Pin_3), U12.2 (GND); no longer R1.2
- net UART4_RX_I2C2: no longer U8.81 (PD0)
- net UART4_TX_I2C2: no longer U8.82 (PD1)
- net USART2_CTS_TELEM1: no longer U8.84 (PD3)
- net USART2_RTS_TELEM1: no longer U8.85 (PD4)
- net USART2_RX_TELEM1: no longer U8.87 (PD6)
- net USART2_TX_TELEM1: no longer U8.86 (PD5)
- net USART3_CTS_TELEM2: no longer U8.58 (PD11)
- net USART3_RTS_TELEM2: no longer U8.59 (PD12)
- net USART3_RX_TELEM2: no longer U8.56 (PD9)
- net USART3_TX_TELEM2: no longer U8.55 (PD8)
- net USB_DM: now also U1.C15 (PA11)
- net USB_DP: now also U1.B15 (PA12)
- net VCC_5V: now also J9.1 (Pin_1), C28.1, J16.1 (Pin_1), U12.1 (IN)
- net VDD_3V3: now also C29.1, J16.4 (Pin_4), J17.2 (Pin_2), U12.5 (OUT)
- net VDD_3V3_SPEKTRUM_POWER_EN: no longer U1.B1 (PE4)
- net VDD_3V3_SENSORS_EN: now reaches U1.A1 (PE3)
- net VDD_3V3_SENSORS_EN: now also U12.3 (EN)
- net USART6_TX_TELEM3/(RC_INPUT): now reaches U1.A7 (PG14)
- net USART6_TX_TELEM3/(RC_INPUT): now also J16.2 (Pin_2)
- net BUZZER_1: now reaches U1.B2 (PE5)
- net BUZZER_1: now also J9.9 (Pin_9)
- net SPI1_DRDY4_ICM20602: now reaches U1.P5 (PC5)
- net SPI1_DRDY4_ICM20602: now also U4.6 (INT)
- net RSSI_IN: now reaches U1.R5 (PB0)
- net RSSI_IN: now also R1.2
- net at R1.1: now also J16.3 (Pin_3)
- no-connect marks 4 -> 5
Other:
- note added: "DSM/SBUS RC"
- note added: "S.BUS out for S.BUS servos"
- moved on the sheet: C1, C18, C19, C2, C3, C4, R6, U11, U4
