File: schematic/_autosave-_autosave-_autosave-_autosave-Test1Kicad.kicad_sch (KiCad schematic)
At the start: 76 parts, among them IC1 BMI055, J1 Power Module 1, J10 CAP & ADC IN, J11 SPI Port, J12 I2C A, J13 FMU PWM OUT, J14 PPM RC, J15 2908-05WB-MG, J16 RC, J17 SBUS, J18 IO/PWM out, J2 Power Module 2, J3 USB, J4 Telemetry 1, J5 Telemetry 2, J6 UART & I2C B, J7 CAN 1, J8 CAN 2, J9 GPS Module, U1 STM32F765IIKx, U10 TJA1051TK-3, U11 LT3080xDD, U12 LP5907MFX-3.3, U13 LP5907MFX-3.3, U3 IST8310, U4 ICM-20602, U5 ICM-20689, U6 MS5611-01BA, U8 STM32F103V8Tx, U9 TJA1051TK-3, Y1 ABM2-8.000MHZ-D4Y-T

Commit message: insert power flags, removed third regulator, rename REG_5V and REG_3V
Parts:
- removed C30, C31: 1uf, symbol Device:C_Small
- removed U13: LP5907MFX-3.3, Package_TO_SOT_SMD:SOT-23-5, symbol Regulator_Linear:LP5907MFX-3.3
Connections:
- net VBUS: no longer U1.E15 (PA9), U1.H13 (VDDUSB)
- net VDD_ports: now also J15.4 (VDD), R10.2, R11.2, R7.2, R8.2, R9.2
- net VCC_5V renamed REG_5V
- removed net VDD_3V3: C13.2, C29.1, J16.4 (Pin_4), U1.F3 (VDD), U1.G13 (VDD), U1.G3 (VDD), U1.J12 (VDD), U1.J13 (VDD), U1.K4 (VDD), U1.N10 (VDD), U1.N8 (VDD), U1.N9 (VDD), U1.P1 (VREF+), U1.R1 (VDDA), U12.5 (OUT), U3.2 (AVDD), U8.100 (VDD), U8.11 (VDD), U8.21 (VREF+), U8.22 (VDDA), U8.28 (VDD), U8.50 (VDD), U8.75 (VDD)
- net VDD_5V_RC_EN: no longer names the net of U1.K13 (PG5)
- net VDD_sensors renamed REG_3V
- net REG_3V: now also C13.2, C29.1, J16.4 (Pin_4), U1.F3 (VDD), U1.P1 (VREF+), U12.5 (OUT), U3.2 (AVDD), U8.11 (VDD), U8.21 (VREF+); no longer C6.2, C8.2, U1.C5 (VDD), U5.13 (VDD)
- new net: C6.2, C8.2, U5.13 (VDD)
- no-connect marks 129 -> 151
Other:
- moved on the sheet: J1, J10, J11, J12, J13, J14, J15, J16, J17, J18, J2, J3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
