File: schematic/_autosave-_autosave-_autosave-_autosave-Test1Kicad.kicad_pcb (KiCad board)
At the start: 2 copper layers, 44 x 84 mm, 75 parts, among them IC1 BMI055, J1 Power Module 1, J10 CAP & ADC IN, J11 SPI Port, J12 I2C A, J13 FMU PWM OUT, J14 PPM RC, J15 2908-05WB-MG, J16 RC, J17 SBUS, J18 IO/PWM out, J2 Power Module 2, J3 USB, J4 Telemetry 1, J5 Telemetry 2, J6 UART & I2C B, J7 CAN 1, J8 CAN 2, J9 GPS Module, U1 STM32F765IIKx, U10 TJA1051TK-3, U11 LT3080xDD, U12 LP5907MFX-3.3, U3 IST8310, U4 ICM-20602, U5 ICM-20689, U6 MS5611-01BA, U8 STM32F103V8Tx, U9 TJA1051TK-3, Y1 ABM2-8.000MHZ-D4Y-T

Commit message: -
Parts:
- moved U8 59.5 mm to (151.5, 81.2)
Changed lines of the file:
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@@
 	(footprint "Package_QFP:LQFP-100_14x14mm_P0.5mm"
 		(layer "F.Cu")
-		(at 94.23 64.88)
+		(at 151.5 81.175)
 		(descr "LQFP, 100 Pin (https://www.nxp.com/docs/en/package-information/SOT407-1.pdf), generated with kicad-footprint-generator ipc_gullwing_generator.py")
 		(tags "LQFP QFP")
