File: project_file/project_file.kicad_sch (KiCad schematic)
At the start: 76 parts, among them IC1 BMI055, J1 Power Module 1, J10 CAP & ADC IN, J11 SPI Port, J12 I2C A, J13 FMU PWM OUT, J14 PPM RC, J15 2908-05WB-MG, J16 RC, J17 SBUS, J18 IO/PWM out, J2 Power Module 2, J3 USB, J4 Telemetry 1, J5 Telemetry 2, J6 UART & I2C B, J7 CAN 1, J8 CAN 2, J9 GPS Module, U1 STM32F765IIKx, U10 TJA1051TK-3, U11 LT3080xDD, U12 LP5907MFX-3.3, U13 LP5907MFX-3.3, U3 IST8310, U4 ICM-20602, U5 ICM-20689, U6 MS5611-01BA, U8 STM32F103V8Tx, U9 TJA1051TK-3, Y1 ABM2-8.000MHZ-D4Y-T

Commit message: Big changes
i removed the second mcu and added in decoupling capacitors and a switch and led so we know when its on
Parts:
- removed U8: STM32F103V8Tx, Package_QFP:LQFP-100_14x14mm_P0.5mm, symbol MCU_ST_STM32F1:STM32F103V8Tx
- added C32, C33, C34, C35, C36, C37, C38, C39, C40, C41: 100nf, Capacitor_SMD:C_0201_0603Metric, symbol Device:C_Small
- added D1: LED, symbol Device:LED
- added R5: 300R, symbol Device:R
- added SW1: SW_Nidec_CAS-120A1, Button_Switch_SMD:Nidec_Copal_CAS-120A, symbol Switch:SW_Nidec_CAS-120A1
- J18: footprint Connector_JST:JST_GH_BM10B-GHS-TBT_1x10-1MP_P1.25mm_Vertical -> Connector_JST:JST_GH_BM08B-GHS-TBT_1x10-1MP_P1.25mm_Vertical
Connections:
- net ADC1_SPARE_1 (3.3V): now also U1.H4 (PH4)
- net ADC1_SPARE_2 (6.6V): now also U1.J4 (PH5)
- net BMS_22.2V: now also SW1.2 (B); no longer C18.1, U11.5 (V_{CONTROL}), U11.7 (IN), U11.8 (IN)
- net CAN1_RX: now also U1.E3 (PI10); no longer U1.D3 (PI9)
- net FMU_CAP1: now also U1.K14 (PG4)
- net FMU_CAP2: now also U1.K15 (PG3)
- net FMU_CAP3: now also U1.D2 (PI8)
- net GND: now also SW1.1 (C)
- net IO_CH1: now also U1.D4 (PI4)
- net IO_CH2: now also U1.C13 (PI3)
- net IO_CH3: now also U1.C14 (PI2)
- net IO_CH4: now also U1.D14 (PI1)
- net IO_CH5: now also U1.B10 (PG10)
- net IO_CH6: now also U1.C10 (PG9)
- net IO_CH7: now also U1.H14 (PG8)
- net IO_CH8: now also U1.J14 (PG7)
- net RC_INPUT (aka PPM_IN): now also U1.C2 (PI7)
- net RSSI_IN: now also U1.C4 (PI5)
- net SBUS_OUT: now also U1.E14 (PI0)
- net SPI1_CS4_BMI055_ACC: now also U1.B9 (PG11); no longer U1.B10 (PG10)
- net SPI1_SCK: now also U1.B8 (PG12); no longer U1.B9 (PG11)
- net SPI5_CS1_EXTERNAL1: now also U1.D3 (PI9); no longer U1.D4 (PI4)
- net SPI5_CS2_EXTERNAL1: now also U1.E4 (PI11); no longer U1.E3 (PI10)
- net TIM1_CH1: now also U1.L15 (PG2)
- net UART8_RX_PX4IO: now also U1.M7 (PG1)
- net UART8_TX_PX4IO: now also U1.N7 (PG0)
- net USART6_TX_TELEM3/(RC_INPUT): now also U1.C3 (PI6)
- net VBUS: now also U1.J15 (PG6)
- net VDD_3V3: now also C32.1, C33.1, C34.1, C35.1, C36.1, C37.1, C38.1, C39.1, C40.1, C41.1; no longer U1.F3 (VDD), U1.G13 (VDD), U1.G3 (VDD), U1.J12 (VDD), U1.J13 (VDD), U1.K4 (VDD), U1.N10 (VDD), U1.N8 (VDD), U1.N9 (VDD), U1.R1 (VDDA)
- new net: C32.2, U1.F3 (VDD)
- new net: C34.2, U1.G13 (VDD)
- new net: C33.2, U1.G3 (VDD)
- new net: C35.2, U1.J12 (VDD)
- new net: C36.2, U1.J13 (VDD)
- new net: C37.2, U1.K4 (VDD)
- new net: C40.2, U1.N10 (VDD)
- new net: C38.2, U1.N8 (VDD)
- new net: C39.2, U1.N9 (VDD)
- new net: C41.2, U1.R1 (VDDA)
- new net: C18.1, R5.2, U11.5 (V_{CONTROL}), U11.7 (IN), U11.8 (IN)
- new net: D1.1 (K), R5.1
- new net: D1.2 (A), SW1.3 (A)
- no-connect marks 129 -> 49
Other:
- moved on the sheet: C28, C29, U12

Commit message: deleted old 22v to 5v regulator
Parts:
- removed C30, C31: 1uf, Capacitor_SMD:C_0603_1608Metric, symbol Device:C_Small
- removed U13: LP5907MFX-3.3, Package_TO_SOT_SMD:SOT-23-5, symbol Regulator_Linear:LP5907MFX-3.3

Commit message: sorted VDD input to sensprs/ports
Parts:
- added C30, C31, C42: 0.1uF, Capacitor_SMD:C_0603_1608Metric, symbol Device:C_Small
- added C43, C44, C45: 100nf, Capacitor_SMD:C_0201_0603Metric, symbol Device:C_Small
- C5: value 0.47uF -> 0.1uF
- J18: footprint Connector_JST:JST_GH_BM08B-GHS-TBT_1x10-1MP_P1.25mm_Vertical -> Connector_JST:JST_GH_BM10B-GHS-TBT_1x10-1MP_P1.25mm_Vertical
Connections:
- net SCL_2 is gone; now on net I2C3_SCL: R4.2, U3.1 (SCL)
- net SDA_2 is gone; now on net I2C3_SDA: R3.2, U3.16 (SDA)
- net VDD is gone; now on net VDD_3V3: R3.1, R4.1
- net VDDIO is gone; now on net VDD_3V3: C26.2, C27.2, U10.5 (VIO), U9.5 (VIO)
- net GND: now also C30.2
- net VDD_3V3: now also C10.2, C11.1, C2.2, C3.1, C4.2, C6.2, C7.1, C8.2, C9.1, IC1.11 (VDDIO), IC1.3 (VDD), J15.4 (VDD), R10.2, R11.2, R7.2, R8.2, R9.2, U3.13 (DVDD), U4.1 (VDDIO), U4.16 (VDD), U5.13 (VDD), U5.8 (VDDIO), U6.1 (VDD), C30.1, C31.2, C42.2, C43.1, C44.1, C45.1
- net I2C3_SDA: now reaches U1.M12 (PH8)
- net I2C3_SCL: now reaches U1.N12 (PH7)
- removed net VDDIO_sensors: C11.1, C3.1, C7.1, IC1.11 (VDDIO), U1.C7 (VDD), U4.1 (VDDIO), U5.8 (VDDIO)
- net VDD_5V_RC_EN: no longer names the net of U1.K13 (PG5)
- removed net VDD_ports: J15.4 (VDD), J9.8 (Pin_8), R10.2, R11.2, R7.2, R8.2, R9.2, U1.C9 (VDD)
- removed net VDD_sensors: C10.2, C2.2, C4.2, C6.2, C8.2, C9.1, IC1.3 (VDD), U1.C5 (VDD), U3.13 (DVDD), U4.16 (VDD), U5.13 (VDD), U6.1 (VDD)
- new net: C45.2, U1.C5 (VDD)
- new net: C44.2, U1.C7 (VDD)
- new net: C43.2, U1.C9 (VDD)
- new net: C31.1, C42.1, J9.8 (Pin_8)
- no-connect marks 49 -> 54
Other:
- moved on the sheet: C12, C13, R3, R4, U3

Commit message: changed JST connectors to pads
Parts:
- removed J1: Power Module 1, Connector_JST:JST_GH_BM06B-GHS-TBT_1x06-1MP_P1.25mm_Vertical, symbol Connector:Conn_01x06_Socket
- removed J10: CAP & ADC IN, Connector_JST:JST_GH_BM08B-GHS-TBT_1x08-1MP_P1.25mm_Vertical, symbol Connector:Conn_01x08_Socket
- removed J11: SPI Port, Connector_JST:JST_GH_BM07B-GHS-TBT_1x07-1MP_P1.25mm_Vertical, symbol Connector:Conn_01x07_Socket
- removed J12: I2C A, Connector_JST:JST_GH_BM04B-GHS-TBT_1x04-1MP_P1.25mm_Vertical, symbol Connector:Conn_01x04_Socket
- removed J13: FMU PWM OUT, Connector_JST:JST_EH_B10B-EH-A_1x10_P2.50mm_Vertical, symbol Connector:Conn_01x10_Socket
- removed J14: PPM RC, Connector_JST:JST_GH_BM03B-GHS-TBT_1x03-1MP_P1.25mm_Vertical, symbol Connector:Conn_01x03_Socket
- removed J16: RC, Connector_JST:JST_GH_BM05B-GHS-TBT_1x05-1MP_P1.25mm_Vertical, symbol Connector:Conn_01x05_Socket
- removed J17: SBUS, Connector_JST:JST_GH_BM03B-GHS-TBT_1x03-1MP_P1.25mm_Vertical, symbol Connector:Conn_01x03_Socket
- removed J18: IO/PWM out, Connector_JST:JST_GH_BM10B-GHS-TBT_1x10-1MP_P1.25mm_Vertical, symbol Connector:Conn_01x10_Socket
- removed J2: Power Module 2, Connector_JST:JST_GH_BM06B-GHS-TBT_1x06-1MP_P1.25mm_Vertical, symbol Connector:Conn_01x06_Socket
- removed J3: USB, Connector_JST:JST_GH_BM04B-GHS-TBT_1x04-1MP_P1.25mm_Vertical, symbol Connector:Conn_01x04_Socket
- removed J4: Telemetry 1, Connector_JST:JST_GH_BM06B-GHS-TBT_1x06-1MP_P1.25mm_Vertical, symbol Connector:Conn_01x06_Socket
- removed J5: Telemetry 2, Connector_JST:JST_GH_BM06B-GHS-TBT_1x06-1MP_P1.25mm_Vertical, symbol Connector:Conn_01x06_Socket
- removed J6: UART & I2C B, Connector_JST:JST_GH_BM06B-GHS-TBT_1x06-1MP_P1.25mm_Vertical, symbol Connector:Conn_01x06_Socket
- removed J9: GPS Module, Connector_JST:JST_GH_BM10B-GHS-TBT_1x10-1MP_P1.25mm_Vertical, symbol Connector:Conn_01x10_Socket
- added J1, J2, J3: Conn_01x01_Socket, Connector_Wire:SolderWirePad_1x01_SMD_5x10mm, symbol Connector:Conn_01x01_Socket
- added J10, J11, J12, J13, J14, J16, J17, J18, J19, J20, J21, J22, J23, J24, J25, J26, J27, J28, J29, J30, J31, J32, J33, J34, J35, J36, J37, J38, J39, J4, J40, J41, J42, J43, J44, J45, J46, J47, J48, J49, J5, J50, J51, J52, J53, J54, J55, J56, J57, J58, J59, J6, J60, J61, J62, J63, J64, J65, J66, J67, J68, J69, J70, J9: Conn_01x01_Socket, Connector_Wire:SolderWirePad_1x01_SMD_1x2mm, symbol Connector:Conn_01x01_Socket
Connections:
- net ADC1_SPARE_1 (3.3V): now also J55.1 (Pin_1)
- net ADC1_SPARE_2 (6.6V): now also J54.1 (Pin_1)
- net BAT1_I: now also J6.1 (Pin_1)
- net BAT1_V: now also J9.1 (Pin_1)
- net BAT2_I: now also J12.1 (Pin_1)
- net BAT2_V: now also J13.1 (Pin_1)
- net BMS_22.2V: now also J10.1 (Pin_1), J11.1 (Pin_1), J4.1 (Pin_1), J5.1 (Pin_1)
- net BUZZER_1: now also J30.1 (Pin_1)
- net FMU_CAP1: now also J59.1 (Pin_1)
- net FMU_CAP2: now also J58.1 (Pin_1)
- net FMU_CAP3: now also J57.1 (Pin_1)
- net FMU_CH1: now also J46.1 (Pin_1)
- net FMU_CH2: now also J45.1 (Pin_1)
- net FMU_CH3: now also J44.1 (Pin_1)
- net FMU_CH4: now also J43.1 (Pin_1)
- net FMU_CH5: now also J42.1 (Pin_1)
- net FMU_CH6: now also J41.1 (Pin_1)
- net FMU_CH7: now also J40.1 (Pin_1)
- net FMU_CH8: now also J39.1 (Pin_1)
- net GND: now also J3.1 (Pin_1)
- net I2C1_SDA_GPS1: now also J33.1 (Pin_1)
- net I2C2_SCL_UART4: now also J28.1 (Pin_1)
- net I2C2_SDA_UART4: now also J29.1 (Pin_1)
- net I2C4_SCL_EXTERNAL2: now also J38.1 (Pin_1)
- net I2C4_SDA_EXTERNAL2: now also J37.1 (Pin_1)
- net IO_CH1: now also J69.1 (Pin_1)
- net IO_CH2: now also J68.1 (Pin_1)
- net IO_CH3: now also J67.1 (Pin_1)
- net IO_CH4: now also J66.1 (Pin_1)
- net IO_CH5: now also J65.1 (Pin_1)
- net IO_CH6: now also J64.1 (Pin_1)
- net IO_CH7: now also J63.1 (Pin_1)
- net IO_CH8: now also J62.1 (Pin_1)
- net RC_INPUT (aka PPM_IN): now also J53.1 (Pin_1)
- net SAFETY_SWITCH_IN: now also J32.1 (Pin_1)
- net SBUS_OUT: now also J70.1 (Pin_1)
- net SPI5_CS1_EXTERNAL1: now also J49.1 (Pin_1)
- net SPI5_CS2_EXTERNAL1: now also J48.1 (Pin_1)
- net SPI5_MISO_EXTERNAL1: now also J51.1 (Pin_1)
- net SPI5_MOSI_EXTERNAL1: now also J50.1 (Pin_1)
- net SPI5_SCK_EXTERNAL1: now also J52.1 (Pin_1)
- net TIM1_CH1: now also J56.1 (Pin_1)
- net UART4_RX_I2C2: now also J27.1 (Pin_1)
- net UART4_TX_I2C2: now also J26.1 (Pin_1)
- net USART1_RX_GPS1: now also J35.1 (Pin_1)
- net USART1_TX_GPS1: now also J36.1 (Pin_1)
- net USART2_CTS_TELEM1: now also J20.1 (Pin_1)
- net USART2_RTS_TELEM1: now also J21.1 (Pin_1)
- net USART2_RX_TELEM1: now also J19.1 (Pin_1)
- net USART2_TX_TELEM1: now also J18.1 (Pin_1)
- net USART3_CTS_TELEM2: now also J24.1 (Pin_1)
- net USART3_RTS_TELEM2: now also J25.1 (Pin_1)
- net USART3_RX_TELEM2: now also J23.1 (Pin_1)
- net USART3_TX_TELEM2: now also J22.1 (Pin_1)
- net USART6_TX_TELEM3/(RC_INPUT): now also J61.1 (Pin_1)
- net USB_DM: now also J16.1 (Pin_1)
- net USB_DP: now also J17.1 (Pin_1)
- net VBUS: now also J14.1 (Pin_1)
- net VCC_5V: now also J2.1 (Pin_1)
- net VDD_3V3: now also J1.1 (Pin_1)
- net at R1.1: now also J60.1 (Pin_1)
- net at C31.1, C42.1: now also J31.1 (Pin_1)
- new net VDD_Servo: J47.1 (Pin_1)
- no-connect marks 54 -> 51
Other:
- note added: "Common GND & Power"
- note added: "UART & I2C B(for additional GPS)"
- note removed: "UART and I2C (for additional GPS)"
- moved on the sheet: R1

Commit message: CAN JST to pads, group pcb components tgt
Parts:
- removed J7: CAN 1, Connector_JST:JST_GH_BM04B-GHS-TBT_1x04-1MP_P1.25mm_Vertical, symbol Connector:Conn_01x04_Socket
- removed J8: CAN 2, Connector_JST:JST_GH_BM04B-GHS-TBT_1x04-1MP_P1.25mm_Vertical, symbol Connector:Conn_01x04_Socket
- added J71, J72, J73, J74, J75, J76: Conn_01x01_Socket, Connector_Wire:SolderWirePad_1x01_SMD_1x2mm, symbol Connector:Conn_01x01_Socket
- D1: footprint (none) -> LED_SMD:LED_0603_1608Metric
- R5: value 300R -> 300; footprint (none) -> Resistor_SMD:R_0603_1608Metric
Connections:
- net GND: now also C20.1, C25.1, R12.2, R13.2, R14.2, R15.2, J72.1 (Pin_1), J73.1 (Pin_1), J75.1 (Pin_1), J76.1 (Pin_1)
- net VCC_5V: now also J71.1 (Pin_1), J74.1 (Pin_1)
Other:
- moved on the sheet: C28
