File: project_file/project_file.kicad_pcb (KiCad board)
At the start: 2 copper layers, 147 parts, among them IC1 BMI055, J1 Conn_01x01_Socket, J10 Conn_01x01_Socket, J11 Conn_01x01_Socket, J12 Conn_01x01_Socket, J13 Conn_01x01_Socket, J14 Conn_01x01_Socket, J15 2908-05WB-MG, J16 Conn_01x01_Socket, J17 Conn_01x01_Socket, J18 Conn_01x01_Socket, J19 Conn_01x01_Socket, J2 Conn_01x01_Socket, J20 Conn_01x01_Socket, J21 Conn_01x01_Socket, J22 Conn_01x01_Socket, J23 Conn_01x01_Socket, J24 Conn_01x01_Socket, J25 Conn_01x01_Socket, J26 Conn_01x01_Socket, J27 Conn_01x01_Socket, J28 Conn_01x01_Socket, J29 Conn_01x01_Socket, J3 Conn_01x01_Socket, J30 Conn_01x01_Socket, J31 Conn_01x01_Socket, J32 Conn_01x01_Socket, J33 Conn_01x01_Socket, J34 Conn_01x01_Socket, J35 Conn_01x01_Socket, J36 Conn_01x01_Socket, J37 Conn_01x01_Socket, J38 Conn_01x01_Socket, J39 Conn_01x01_Socket, J4 Conn_01x01_Socket, J40 Conn_01x01_Socket, J41 Conn_01x01_Socket, J42 Conn_01x01_Socket, J43 Conn_01x01_Socket, J44 Conn_01x01_Socket, J45 Conn_01x01_Socket, J46 Conn_01x01_Socket, J47 Conn_01x01_Socket, J48 Conn_01x01_Socket, J49 Conn_01x01_Socket, J5 Conn_01x01_Socket, J50 Conn_01x01_Socket, J51 Conn_01x01_Socket, J52 Conn_01x01_Socket, J53 Conn_01x01_Socket, J54 Conn_01x01_Socket, J55 Conn_01x01_Socket, J56 Conn_01x01_Socket, J57 Conn_01x01_Socket, J58 Conn_01x01_Socket, J59 Conn_01x01_Socket, J6 Conn_01x01_Socket, J60 Conn_01x01_Socket, J61 Conn_01x01_Socket, J62 Conn_01x01_Socket, J63 Conn_01x01_Socket, J64 Conn_01x01_Socket, J65 Conn_01x01_Socket, J66 Conn_01x01_Socket, J67 Conn_01x01_Socket, J68 Conn_01x01_Socket, J69 Conn_01x01_Socket, J70 Conn_01x01_Socket, J71 Conn_01x01_Socket, J72 Conn_01x01_Socket, J73 Conn_01x01_Socket, J74 Conn_01x01_Socket, J75 Conn_01x01_Socket, J76 Conn_01x01_Socket, J9 Conn_01x01_Socket, SW1 SW_Nidec_CAS-120A1, U1 STM32F765IIKx, U10 TJA1051TK-3, U11 LT3080xDD, U12 LP5907MFX-3.3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

Commit message: -
Parts:
- moved R8 114.7 mm to (214.7, 90.1)
- moved R9 114.7 mm to (208.7, 97.5)
- moved J15 114.7 mm to (213.5, 78.5)
- moved R10 114.7 mm to (222.3, 98.3)
- moved R11 114.7 mm to (216.3, 98.3)
- moved R7 114.7 mm to (211.7, 93.9)
- moved U1 111.7 mm to (180.1, 74.7)
- moved J74 76.3 mm to (91.8, 141.0)
- moved J76 74.8 mm to (108.6, 142.0)
- moved J75 74.3 mm to (111.8, 142.0)
- moved J73 7.84 mm to (117.2, 172.4)
- moved J72 3.74 mm to (114.4, 172.2)
- moved J71 2.43 mm to (98.2, 181.2)
Changed lines of the file:
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@@
 	(footprint "Resistor_SMD:R_0603_1608Metric"
 		(layer "F.Cu")
-		(at 95.575 116.2)
+		(at 208.715 97.5)
 		(descr "Resistor SMD 0603 (1608 Metric), square (rectangular) end terminal, IPC_7351 nominal, (Body size source: IPC-SM-782 page 72, https://www.pcb-3d.com/wordpress/wp-content/uploads/ipc-sm-782a_amendment_1_and_2.pdf), generated with kicad-footprint-generator")
 		(tags "resistor")
@@
 	(footprint "Resistor_SMD:R_0603_1608Metric"
 		(layer "F.Cu")
-		(at 101.55 108.8)
+		(at 214.69 90.1)
 		(descr "Resistor SMD 0603 (1608 Metric), square (rectangular) end terminal, IPC_7351 nominal, (Body size source: IPC-SM-782 page 72, https://www.pcb-3d.com/wordpress/wp-content/uploads/ipc-sm-782a_amendment_1_and_2.pdf), generated with kicad-footprint-generator")
 		(tags "resistor")
@@
 	(footprint "Connector_Wire:SolderWirePad_1x01_SMD_1x2mm"
 		(layer "F.Cu")
-		(at 98.6 183.6)
+		(at 98.2 181.2)
 		(descr "Wire Pad, Square, SMD Pad,  1mm x 2mm,")
 		(tags "MesurementPoint Square SMDPad 1mmx2mm ")
@@
 			(at 0 2.54 0)
 			(layer "F.Fab")
+			(hide yes)
 			(effects
 				(font
@@
 	(footprint "Resistor_SMD:R_0603_1608Metric"
 		(layer "F.Cu")
-		(at 109.125 117 180)
+		(at 222.265 98.3 180)
 		(descr "Resistor SMD 0603 (1608 Metric), square (rectangular) end terminal, IPC_7351 nominal, (Body size source: IPC-SM-782 page 72, https://www.pcb-3d.com/wordpress/wp-content/uploads/ipc-sm-782a_amendment_1_and_2.pdf), generated with kicad-footprint-generator")
 		(tags "resistor")
@@
 	(footprint "Connector_Wire:SolderWirePad_1x01_SMD_1x2mm"
 		(layer "F.Cu")
-		(at 118.16 67.8)
+		(at 108.6 142)
 		(descr "Wire Pad, Square, SMD Pad,  1mm x 2mm,")
 		(tags "MesurementPoint Square SMDPad 1mmx2mm ")
@@
 			(at 0 2.54 0)
 			(layer "F.Fab")
+			(hide yes)
 			(effects
 				(font
@@
 	(footprint "Connector_Wire:SolderWirePad_1x01_SMD_1x2mm"
 		(layer "F.Cu")
-		(at 113.44 67.8)
+		(at 91.8 141)
 		(descr "Wire Pad, Square, SMD Pad,  1mm x 2mm,")
 		(tags "MesurementPoint Square SMDPad 1mmx2mm ")
@@
 			(at 0 2.54 0)
 			(layer "F.Fab")
+			(hide yes)
 			(effects
 				(font
@@
 	(footprint "Resistor_SMD:R_0603_1608Metric"
 		(layer "F.Cu")
-		(at 103.125 117 180)
+		(at 216.265 98.3 180)
 		(descr "Resistor SMD 0603 (1608 Metric), square (rectangular) end terminal, IPC_7351 nominal, (Body size source: IPC-SM-782 page 72, https://www.pcb-3d.com/wordpress/wp-content/uploads/ipc-sm-782a_amendment_1_and_2.pdf), generated with kicad-footprint-generator")
 		(tags "resistor")
@@
 	(footprint "Package_BGA:UFBGA-201_10x10mm_Layout15x15_P0.65mm"
 		(layer "F.Cu")
-		(at 68.4 74.1)
+		(at 180.1 74.7)
 		(descr "UFBGA-201, 10.0x10.0mm, 201 Ball, 15x15 Layout, 0.65mm Pitch, http://www.st.com/resource/en/datasheet/stm32f207vg.pdf#page=166")
 		(tags "BGA 201 0.65")
@@
 	(footprint "Connector_Wire:SolderWirePad_1x01_SMD_1x2mm"
 		(layer "F.Cu")
-		(at 118 180.2)
+		(at 117.2 172.4)
 		(descr "Wire Pad, Square, SMD Pad,  1mm x 2mm,")
 		(tags "MesurementPoint Square SMDPad 1mmx2mm ")
@@
 			(at 0 2.54 0)
 			(layer "F.Fab")
+			(hide yes)
 			(effects
 				(font
@@
 	(footprint "2908-05WB-MG:3M_2908-05WB-MG"
 		(layer "F.Cu")
-		(at 100.4 97.2)
+		(at 213.54 78.5)
 		(property "Reference" "J15"
 			(at -8.27711 3.72596 180)
@@
 			(polygon
 				(pts
-					(xy 107.05387 92.2) (xy 107.65 92.2) (xy 107.65 105.1046) (xy 107.05387 105.1046)
+					(xy 220.19387 73.5) (xy 220.79 73.5) (xy 220.79 86.4046) (xy 220.19387 86.4046)
 				)
 			)
@@
 			(polygon
 				(pts
-					(xy 107.05739 92.21) (xy 107.65 92.21) (xy 107.65 105.10878) (xy 107.05739 105.10878)
+					(xy 220.19739 73.51) (xy 220.79 73.51) (xy 220.79 86.40878) (xy 220.19739 86.40878)
 				)
 			)
@@
 	(footprint "Connector_Wire:SolderWirePad_1x01_SMD_1x2mm"
 		(layer "F.Cu")
-		(at 118 173.2)
+		(at 114.4 172.2)
 		(descr "Wire Pad, Square, SMD Pad,  1mm x 2mm,")
 		(tags "MesurementPoint Square SMDPad 1mmx2mm ")
@@
 			(at 0 2.54 0)
 			(layer "F.Fab")
+			(hide yes)
 			(effects
 				(font
@@
 	(footprint "Resistor_SMD:R_0603_1608Metric"
 		(layer "F.Cu")
-		(at 98.55 112.6)
+		(at 211.69 93.9)
 		(descr "Resistor SMD 0603 (1608 Metric), square (rectangular) end terminal, IPC_7351 nominal, (Body size source: IPC-SM-782 page 72, https://www.pcb-3d.com/wordpress/wp-content/uploads/ipc-sm-782a_amendment_1_and_2.pdf), generated with kicad-footprint-generator")
 		(tags "resistor")
@@
 	(footprint "Connector_Wire:SolderWirePad_1x01_SMD_1x2mm"
 		(layer "F.Cu")
-		(at 115.8 67.8)
+		(at 111.8 142)
 		(descr "Wire Pad, Square, SMD Pad,  1mm x 2mm,")
 		(tags "MesurementPoint Square SMDPad 1mmx2mm ")
@@
 			(at 0 2.54 0)
 			(layer "F.Fab")
+			(hide yes)
 			(effects
 				(font
